File: dohome_switch.sch (KiCad schematic (older format))
At the start: 25 parts, among them P1 FTDI, P2 CONN_02X09, Q1 BSS138, Q2 BSS138, SW1 RST/PRG, U1 RT9013-33GB, U2 ESP-12E, U3 WS2812B

Commit message: CODE: new version with ftdi
Parts:
- removed C3: 0.1uF, Capacitors_SMD:C_0805_HandSoldering, symbol C_Small
- removed C5: 2u2, Capacitors_SMD:C_0805_HandSoldering, symbol C_Small
- removed Q1, Q2: BSS138, TO_SOT_Packages_SMD:SOT-23, symbol BSS138
- removed R6: 470k, Resistors_SMD:R_0805_HandSoldering, symbol R_Small
- removed R7: 100k, Resistors_SMD:R_0805_HandSoldering, symbol R_Small
- P1: footprint Pin_Headers:Pin_Header_Straight_1x06 -> Socket_Strips:Socket_Strip_Straight_1x06_Pitch2.54mm
- P2: value CONN_02X09 -> CONN_02X07; footprint Pin_Headers:Pin_Header_Straight_2x08 -> Pin_Headers:Pin_Header_Angled_2x07_Pitch2.54mm; symbol CONN_02X08 -> CONN_02X07
- U1: symbol RT9013-33GB -> RT9013-33GB-RESCUE-dohome_switch
- U2: symbol ESP-12E -> ESP-12E-RESCUE-dohome_switch
Connections:
- net +3V3: now also P1.1 (P1), P2.13 (P13); no longer P1.3 (P3), P2.2 (P2)
- net +5V: now also P2.14 (P14); no longer P2.1 (P1)
- net A0: now also P2.8 (P8); no longer P2.14 (P14)
- net GPIO0: now also P1.2 (P2), P2.4 (P4); no longer P2.7 (P7)
- net GPIO10: now also P2.7 (P7)
- net GPIO12: now also P2.11 (P11); no longer P2.8 (P8)
- net GPIO13: now also P2.12 (P12); no longer P2.6 (P6)
- net GPIO15: now also P2.2 (P2); no longer P2.4 (P4)
- net GPIO16: now also P2.9 (P9); no longer P2.12 (P12)
- net GPIO2: now also P2.3 (P3); no longer P2.5 (P5)
- net GPIO4: now also P2.5 (P5); no longer P2.9 (P9)
- net GPIO5: now also P2.6 (P6); no longer P2.11 (P11)
- net RESET: now also P1.6 (P6); no longer P2.16 (P16)
- net RXD: now also P1.3 (P3); no longer P1.4 (P4), P2.13 (P13)
- net TXD: now also P1.4 (P4); no longer P1.5 (P5), P2.15 (P15)
- net GND: now reaches U2.9 (GND)
- net GND: now also C1.2, C2.2, C4.2, C6.2, C7.2, P1.5 (P5), P2.1 (P1), R1.2, R10.2, R9.2, SW1.1, U1.2 (GND), U3.3 (VSS)
- no-connect marks 8 -> 5
Other:
- moved on the sheet: P1, SW1

Commit message: CODE: Without lines
Parts:
- removed SW1: RST/PRG, Buttons_Switches_SMD:SW_SPST_TL3342, symbol SW_Push
- added JP1: JP1, Pin_Headers:Pin_Header_Straight_1x02_Pitch2.54mm, symbol Jumper_NC_Small
Connections:
- net +3V3: no longer P1.1 (P1)
- net +5V renamed PWR
- net PWR: now also P1.1 (P1), JP1.1; no longer P2.14 (P14)
- new net: JP1.2, P2.14 (P14)
Other:
- note removed: "RST/PRG button"
Changed lines of the file:
@@
-$EndComp
-$Comp
-L +5V #PWR01
-U 1 1 58EF97BA
-P 800 750
-F 0 "#PWR01" H 800 600 50  0001 C CNN
-F 1 "+5V" H 800 890 50  0000 C CNN
-F 2 "" H 800 750 50  0001 C CNN
-F 3 "" H 800 750 50  0000 C CNN
-	1    800  750
-	1    0    0    -1
 $EndComp
 $Comp
@@
 $EndComp
 $Comp
-L GND #PWR02
+L GND #PWR01
 U 1 1 58EF9890
 P 900 1000
-F 0 "#PWR02" H 900 750 50  0001 C CNN
+F 0 "#PWR01" H 900 750 50  0001 C CNN
 F 1 "GND" H 1100 900 50  0000 C CNN
 F 2 "" H 900 1000 50  0001 C CNN
@@
 $EndComp
 $Comp
-L GND #PWR03
+L GND #PWR02
 U 1 1 58EFA08B
 P 1000 1550
-F 0 "#PWR03" H 1000 1300 50  0001 C CNN
+F 0 "#PWR02" H 1000 1300 50  0001 C CNN
 F 1 "GND" H 1000 1400 50  0000 C CNN
 F 2 "" H 1000 1550 50  0001 C CNN
@@
 $EndComp
 $Comp
-L GND #PWR04
+L GND #PWR03
 U 1 1 58EFA571
 P 1700 1550
-F 0 "#PWR04" H 1700 1300 50  0001 C CNN
+F 0 "#PWR03" H 1700 1300 50  0001 C CNN
 F 1 "GND" H 1700 1400 50  0000 C CNN
 F 2 "" H 1700 1550 50  0001 C CNN
@@
 $EndComp
 $Comp
-L GND #PWR05
+L GND #PWR04
 U 1 1 58EFA62B
 P 2300 1000
-F 0 "#PWR05" H 2300 750 50  0001 C CNN
+F 0 "#PWR04" H 2300 750 50  0001 C CNN
 F 1 "GND" H 2300 850 50  0000 C CNN
 F 2 "" H 2300 1000 50  0001 C CNN
@@
 $EndComp
 $Comp
-L +3.3V #PWR06
+L +3.3V #PWR05
 U 1 1 58EFA721
 P 2550 800
-F 0 "#PWR06" H 2550 650 50  0001 C CNN
+F 0 "#PWR05" H 2550 650 50  0001 C CNN
 F 1 "+3.3V" H 2550 940 50  0000 C CNN
 F 2 "" H 2550 800 50  0001 C CNN
@@
 GPIO0
 $Comp
-L +3.3V #PWR07
+L +3.3V #PWR06
 U 1 1 58EFBAAC
 P 4150 4050
-F 0 "#PWR07" H 4150 3900 50  0001 C CNN
+F 0 "#PWR06" H 4150 3900 50  0001 C CNN
 F 1 "+3.3V" V 4050 4150 50  0000 C CNN
 F 2 "" H 4150 4050 50  0001 C CNN
@@
 	1    5800 3650
 	1    0    0    -1
-$EndComp
-$Comp
-L GND #PWR08
-U 1 1 58EFE830
-P 3900 900
-F 0 "#PWR08" H 3900 650 50  0001 C CNN
-F 1 "GND" H 3900 950 50  0000 C CNN
-F 2 "" H 3900 900 50  0001 C CNN
-F 3 "" H 3900 900 50  0000 C CNN
-	1    3900 900
-	1    0    0    -1
-$EndComp
-Text Label 4050 1300 2    60   ~ 0
-RESET
-Text Notes 3950 1850 2    60   ~ 0
-RST/PRG button
-$Comp
-L SW_Push SW1
-U 1 1 58F0807A
-P 4550 1100
-F 0 "SW1" H 4600 1200 50  0000 L CNN
-F 1 "RST/PRG" H 4550 1040 50  0000 C CNN
-F 2 "Buttons_Switches_SMD:SW_SPST_TL3342" V 4450 1400 50  0001 C CNN
-F 3 "" H 4550 1300 50  0000 C CNN
-	1    4550 1100
-	0    1    1    0
 $EndComp
 Text Label 4900 3450 2    60   ~ 0
@@
 GPIO15
 $Comp
-L GND #PWR09
+L GND #PWR07
 U 1 1 58F0FDB3
 P 6700 4050
-F 0 "#PWR09" H 6700 3800 50  0001 C CNN
+F 0 "#PWR07" H 6700 3800 50  0001 C CNN
 F 1 "GND" H 6700 3900 50  0000 C CNN
 F 2 "" H 6700 4050 50  0001 C CNN
@@
 $EndComp
 $Comp
-L GND #PWR010
+L GND #PWR08
 U 1 1 58F12850
 P 850 3400
-F 0 "#PWR010" H 850 3150 50  0001 C CNN
+F 0 "#PWR08" H 850 3150 50  0001 C CNN
 F 1 "GND" H 850 3250 50  0000 C CNN
 F 2 "" H 850 3400 50  0001 C CNN
@@
 $EndComp
 $Comp
-L GND #PWR011
+L GND #PWR09
 U 1 1 58F12DBE
 P 4450 4250
-F 0 "#PWR011" H 4450 4000 50  0001 C CNN
+F 0 "#PWR09" H 4450 4000 50  0001 C CNN
 F 1 "GND" H 4450 4100 50  0000 C CNN
 F 2 "" H 4450 4250 50  0001 C CNN
@@
 $EndComp
 $Comp
-L +3.3V #PWR012
+L +3.3V #PWR010
 U 1 1 58F1362B
 P 850 2250
-F 0 "#PWR012" H 850 2100 50  0001 C CNN
+F 0 "#PWR010" H 850 2100 50  0001 C CNN
 F 1 "+3.3V" H 850 2390 50  0000 C CNN
 F 2 "" H 850 2250 50  0001 C CNN
@@
 Pull-up/down resistors
 $Comp
-L GND #PWR013
+L GND #PWR011
 U 1 1 58F1572A
 P 5800 1700
-F 0 "#PWR013" H 5800 1450 50  0001 C CNN
+F 0 "#PWR011" H 5800 1450 50  0001 C CNN
 F 1 "GND" H 5800 1550 50  0000 C CNN
 F 2 "" H 5800 1700 50  0001 C CNN
@@
 $EndComp
 $Comp
-L GND #PWR014
+L GND #PWR012
 U 1 1 58F162FD
 P 8750 1400
-F 0 "#PWR014" H 8750 1150 50  0001 C CNN
+F 0 "#PWR012" H 8750 1150 50  0001 C CNN
 F 1 "GND" H 8750 1250 50  0000 C CNN
 F 2 "" H 8750 1400 50  0001 C CNN
 F 3 "" H 8750 1400 50  0000 C CNN
 	1    8750 1400
-	1    0    0    -1
-$EndComp
-$Comp
-L +5V #PWR015
-U 1 1 58F16480
-P 7350 950
-F 0 "#PWR015" H 7350 800 50  0001 C CNN
-F 1 "+5V" H 7350 1090 50  0000 C CNN
-F 2 "" H 7350 950 50  0001 C CNN
-F 3 "" H 7350 950 50  0000 C CNN
-	1    7350 950
 	1    0    0    -1
 $EndComp
@@
 NoConn ~ 7850 1300
 $Comp
-L GND #PWR016
+L GND #PWR013
 U 1 1 58F17315
 P 7650 1350
-F 0 "#PWR016" H 7650 1100 50  0001 C CNN
+F 0 "#PWR013" H 7650 1100 50  0001 C CNN
 F 1 "GND" H 7650 1200 50  0000 C CNN
 F 2 "" H 7650 1350 50  0001 C CNN
@@
 RGB LED
 $Comp
-L GND #PWR017
+L GND #PWR014
 U 1 1 58F192EC
 P 1750 4150
-F 0 "#PWR017" H 1750 3900 50  0001 C CNN
+F 0 "#PWR014" H 1750 3900 50  0001 C CNN
 F 1 "GND" H 1750 4000 50  0000 C CNN
 F 2 "" H 1750 4150 50  0001 C CNN
@@
 Text Label 1350 4250 0    60   ~ 0
 TXD
-$Comp
-L +3.3V #PWR018
-U 1 1 58F19880
-P 1750 4550
-F 0 "#PWR018" H 1750 4400 50  0001 C CNN
-F 1 "+3.3V" H 1750 4690 50  0000 C CNN
-F 2 "" H 1750 4550 50  0001 C CNN
-F 3 "" H 1750 4550 50  0000 C CNN
-	1    1750 4550
-	1    0    0    -1
-$EndComp
 Text Notes 1700 5050 0    60   ~ 0
 FTDI
@@
 $EndComp
 $Comp
-L GND #PWR019
+L GND #PWR015
 U 1 1 58F1AAD4
 P 2500 6950
-F 0 "#PWR019" H 2500 6700 50  0001 C CNN
+F 0 "#PWR015" H 2500 6700 50  0001 C CNN
 F 1 "GND" H 2500 6800 50  0000 C CNN
 F 2 "" H 2500 6950 50  0001 C CNN
@@
 GPIO5
 $Comp
-L +3.3V #PWR020
+L +3.3V #PWR016
 U 1 1 58F1ADB5
 P 2750 6250
-F 0 "#PWR020" H 2750 6100 50  0001 C CNN
+F 0 "#PWR016" H 2750 6100 50  0001 C CNN
 F 1 "+3.3V" H 2750 6390 50  0000 C CNN
 F 2 "" H 2750 6250 50  0001 C CNN
@@
 GPIO10
 Wire Wire Line
-	3900 900  4550 900
-Wire Wire Line
-	4050 1300 4550 1300
-Wire Wire Line
 	5800 1500 5800 1700
 Wire Wire Line
-	1750 4550 1350 4550
-Wire Wire Line
 	1350 4150 1750 4150
-$Comp
-L +5V #PWR021
-U 1 1 59142707
-P 1800 6250
-F 0 "#PWR021" H 1800 6100 50  0001 C CNN
-F 1 "+5V" H 1800 6390 50  0000 C CNN
-F 2 "" H 1800 6250 50  0000 C CNN
-F 3 "" H 1800 6250 50  0000 C CNN
-	1    1800 6250
-	1    0    0    -1
-$EndComp
-Wire Wire Line
-	800  800  800  750
-$Comp
-L +5V #PWR022
-U 1 1 5914542D
-P 800 1300
-F 0 "#PWR022" H 800 1150 50  0001 C CNN
-F 1 "+5V" H 800 1440 50  0000 C CNN
-F 2 "" H 800 1300 50  0000 C CNN
-F 3 "" H 800 1300 50  0000 C CNN
-	1    800  1300
-	1    0    0    -1
-$EndComp
+Wire Wire Line
+	800  750  800  1300
+$Comp
+L Jumper_NC_Small JP1
+U 1 1 59149387
+P 1800 6150
+F 0 "JP1" V 1750 6250 50  0000 C CNN
+F 1 "JP1" V 1850 6050 50  0000 C CNN
+F 2 "Pin_Headers:Pin_Header_Straight_1x02_Pitch2.54mm" H 1800 6150 50  0001 C CNN
+F 3 "" H 1800 6150 50  0000 C CNN
+	1    1800 6150
+	0    1    1    0
+$EndComp
+Text Label 1800 5900 2    60   ~ 0
+PWR
+Wire Wire Line
+	1800 6050 1800 5900
+Connection ~ 800  800
+Text Label 800  750  2    60   ~ 0
+PWR
+Text Label 7350 950  2    60   ~ 0
+PWR
+Text Label 1350 4550 0    60   ~ 0
+PWR
 $EndSCHEMATC

Commit message: CODE: first version
Changed lines of the file:
@@
 L GND #PWR015
 U 1 1 58F1AAD4
-P 2500 6950
-F 0 "#PWR015" H 2500 6700 50  0001 C CNN
-F 1 "GND" H 2500 6800 50  0000 C CNN
-F 2 "" H 2500 6950 50  0001 C CNN
-F 3 "" H 2500 6950 50  0000 C CNN
-	1    2500 6950
+P 2800 7000
+F 0 "#PWR015" H 2800 6750 50  0001 C CNN
+F 1 "GND" H 2800 6850 50  0000 C CNN
+F 2 "" H 2800 7000 50  0001 C CNN
+F 3 "" H 2800 7000 50  0000 C CNN
+	1    2800 7000
 	1    0    0    -1
 $EndComp
@@
 Text Label 1350 4550 0    60   ~ 0
 PWR
+Wire Wire Line
+	2500 6950 2800 6950
+Wire Wire Line
+	2800 6950 2800 7000
 $EndSCHEMATC
